File: design/electrical/communication_system.sch (KiCad schematic (older format))
At the start: 18 parts, among them P1a SMA, P2a CONN_01X02, U1a AS193-73, U2a TPS2024DR

Commit message: Finished schematics
Parts:
- R1a: renamed from R?; value R -> 0.1
- R2a: renamed from R?; value R -> 10k
Changed lines of the file:
@@
 -ANT_DEPLOY
 $Comp
-L R R?
+L R R2a
 U 1 1 589B7789
 P 1500 3500
-F 0 "R?" V 1580 3500 50  0000 C CNN
-F 1 "R" V 1500 3500 50  0000 C CNN
+F 0 "R2a" V 1580 3500 50  0000 C CNN
+F 1 "10k" V 1500 3500 50  0000 C CNN
 F 2 "" V 1430 3500 50  0001 C CNN
 F 3 "" H 1500 3500 50  0001 C CNN
@@
 $EndComp
 $Comp
-L R R?
+L R R1a
 U 1 1 589B7AC8
 P 2800 3250
-F 0 "R?" V 2880 3250 50  0000 C CNN
-F 1 "R" V 2800 3250 50  0000 C CNN
+F 0 "R1a" V 2880 3250 50  0000 C CNN
+F 1 "0.1" V 2800 3250 50  0000 C CNN
 F 2 "" V 2730 3250 50  0001 C CNN
 F 3 "" H 2800 3250 50  0001 C CNN
