File: design/electrical/high_power_amplifier_module.sch (KiCad schematic (older format))
At the start: 0 parts

Commit message: Finished schematics
Parts:
- added C1g, C3g, C5g, C7g: 10nF, symbol C
- added C2g, C4g, C6g, C8g: 10uF, symbol C
- added R1g, R3g: 10k, symbol R
- added R2g: 1.1k, symbol R
- added U1g: MAX893L, symbol MAX893L
- added U2g: SKY65116, symbol SKY65116
- added U3g: TMP20AIDRL, symbol TMP20AIDRL
Connections:
- net -HPA_ON: now also R1g.2, U1g.3 (!ON)
- net HPAM_EN: now also C1g.1, C2g.1, R3g.1, U2g.11 (VCNT)
- net RFIN: now also U2g.2 (RFIN)
- net RFOUT: now also U2g.8 (RFOUT)
- net TEMPOUT: now also U3g.3 (Vout)
- new net: R2g.1, U1g.5 (SET)
- new net +3V3: U3g.4 (Vdd)
- new net GND: C1g.2, C2g.2, C3g.2, C4g.2, C5g.2, C6g.2, C7g.2, C8g.2, R2g.2, R3g.2, U1g.4 (GND), U2g.1 (GND), U2g.3 (GND), U2g.5 (GND), U2g.6 (GND), U2g.7 (GND), U2g.9 (GND), U3g.2 (GND), U3g.6 (GND)
- new net VCC_HPA: C3g.1, C4g.1, C5g.1, C6g.1, C7g.1, C8g.1, U1g.6 (OUT), U1g.7 (OUT), U2g.10 (VCC2), U2g.12 (VREF), U2g.4 (VCC1)
- new net VCC_RF: R1g.1, U1g.1 (IN), U1g.2 (IN)
- no-connect marks 0 -> 1
