File: design/electrical/memory_module.sch (KiCad schematic (older format))
At the start: 0 parts

Commit message: Finished schematics
Parts:
- added C1d: 0.1uF, symbol C
- added U1d: IS62WV5128BLL-55TLI-TR, symbol IS62WV5128BLL-55TLI-TR
Connections:
- net -MEM_CE: now also U1d.30 (!CS1)
- net -MEM_OE: now also U1d.32 (!OE)
- net -MEM_WE: now also U1d.5 (!WE)
- net a0: now also U1d.20 (A0)
- net a1: now also U1d.19 (A1)
- net a10: now also U1d.31 (A10)
- net a11: now also U1d.1 (A11)
- net a12: now also U1d.12 (A12)
- net a13: now also U1d.4 (A13)
- net a14: now also U1d.11 (A14)
- net a15: now also U1d.7 (A15)
- net a16: now also U1d.10 (A16)
- net a17: now also U1d.9 (A17)
- net a18: now also U1d.6 (A18)
- net a2: now also U1d.18 (A2)
- net a3: now also U1d.17 (A3)
- net a4: now also U1d.16 (A4)
- net a5: now also U1d.15 (A5)
- net a6: now also U1d.14 (A6)
- net a7: now also U1d.13 (A7)
- net a8: now also U1d.3 (A8)
- net a9: now also U1d.2 (A9)
- net d0: now also U1d.21 (I/O0)
- net d1: now also U1d.22 (I/O1)
- net d2: now also U1d.23 (I/O2)
- net d3: now also U1d.25 (I/O3)
- net d4: now also U1d.26 (I/O4)
- net d5: now also U1d.27 (I/O5)
- net d6: now also U1d.28 (I/O6)
- net d7: now also U1d.29 (I/O7)
- new net +3V3: C1d.1, U1d.8 (VDD)
- new net GND: C1d.2, U1d.24 (GND)
Changed lines of the file:
@@
 $Descr A4 11693 8268
 encoding utf-8
-Sheet 5 7
+Sheet 6 7
 Title ""
 Date ""
@@
 Comment4 ""
 $EndDescr
-Text HLabel 2450 2300 0    60   Input ~ 0
+Text HLabel 5750 3050 2    60   Input ~ 0
 -MEM_CE
-Text HLabel 2450 2600 0    60   Input ~ 0
+Text HLabel 5750 2850 2    60   Input ~ 0
 -MEM_OE
-Text HLabel 2400 2900 0    60   Input ~ 0
+Text HLabel 4800 3250 0    60   Input ~ 0
 -MEM_WE
-Text HLabel 2500 4100 0    60   Input ~ 0
+Text HLabel 5750 3950 2    60   Input ~ 0
 d0
-Text HLabel 2500 4350 0    60   Input ~ 0
+Text HLabel 5750 3850 2    60   Input ~ 0
 d1
-Text HLabel 2500 4550 0    60   Input ~ 0
+Text HLabel 5750 3750 2    60   Input ~ 0
 d2
-Text HLabel 2500 4700 0    60   Input ~ 0
+Text HLabel 5750 3550 2    60   Input ~ 0
 d3
-Text HLabel 2500 4900 0    60   Input ~ 0
+Text HLabel 5750 3450 2    60   Input ~ 0
 d4
-Text HLabel 2500 5050 0    60   Input ~ 0
+Text HLabel 5750 3350 2    60   Input ~ 0
 d5
-Text HLabel 2500 5250 0    60   Input ~ 0
+Text HLabel 5750 3250 2    60   Input ~ 0
 d6
-Text HLabel 2500 5450 0    60   Input ~ 0
+Text HLabel 5750 3150 2    60   Input ~ 0
 d7
-Text HLabel 3750 2250 0    60   Input ~ 0
+Text HLabel 5750 4050 2    60   Input ~ 0
 a0
-Text HLabel 3750 2350 0    60   Input ~ 0
+Text HLabel 5750 4150 2    60   Input ~ 0
 a1
-Text HLabel 3750 2450 0    60   Input ~ 0
+Text HLabel 5750 4250 2    60   Input ~ 0
 a2
-Text HLabel 3700 2600 0    60   Input ~ 0
+Text HLabel 5750 4350 2    60   Input ~ 0
 a3
-Text HLabel 3700 2750 0    60   Input ~ 0
+Text HLabel 4800 4350 0    60   Input ~ 0
 a4
-Text HLabel 3750 2900 0    60   Input ~ 0
+Text HLabel 4800 4250 0    60   Input ~ 0
 a5
-Text HLabel 3750 3050 0    60   Input ~ 0
+Text HLabel 4800 4150 0    60   Input ~ 0
 a6
-Text HLabel 3700 3200 0    60   Input ~ 0
+Text HLabel 4800 4050 0    60   Input ~ 0
 a7
-Text HLabel 3700 3350 0    60   Input ~ 0
+Text HLabel 4800 3050 0    60   Input ~ 0
 a8
-Text HLabel 3700 3500 0    60   Input ~ 0
+Text HLabel 4800 2950 0    60   Input ~ 0
 a9
-Text HLabel 3700 3650 0    60   Input ~ 0
+Text HLabel 5750 2950 2    60   Input ~ 0
 a10
-Text HLabel 3700 3800 0    60   Input ~ 0
+Text HLabel 4800 2850 0    60   Input ~ 0
 a11
-Text HLabel 3800 3950 0    60   Input ~ 0
+Text HLabel 4800 3950 0    60   Input ~ 0
 a12
-Text HLabel 3700 4100 0    60   Input ~ 0
+Text HLabel 4800 3150 0    60   Input ~ 0
 a13
-Text HLabel 3700 4300 0    60   Input ~ 0
+Text HLabel 4800 3850 0    60   Input ~ 0
 a14
-Text HLabel 3700 4500 0    60   Input ~ 0
+Text HLabel 4800 3450 0    60   Input ~ 0
 a15
-Text HLabel 3700 4650 0    60   Input ~ 0
+Text HLabel 4800 3750 0    60   Input ~ 0
 a16
-Text HLabel 3700 4850 0    60   Input ~ 0
+Text HLabel 4800 3650 0    60   Input ~ 0
 a17
-Text HLabel 3750 5000 0    60   Input ~ 0
+Text HLabel 4800 3350 0    60   Input ~ 0
 a18
+$Comp
+L IS62WV5128BLL-55TLI-TR U1d
+U 1 1 5892A45F
+P 5300 3550
+F 0 "U1d" H 5300 4400 60  0000 C CNN
+F 1 "IS62WV5128BLL-55TLI-TR" H 5300 2600 60  0000 C CNN
+F 2 "" H 5300 3600 60  0001 C CNN
+F 3 "" H 5300 3600 60  0001 C CNN
+	1    5300 3550
+	1    0    0    -1
+$EndComp
+$Comp
+L GND #PWR?
+U 1 1 5892A54C
+P 4350 3950
+F 0 "#PWR?" H 4350 3700 50  0001 C CNN
+F 1 "GND" H 4350 3800 50  0000 C CNN
+F 2 "" H 4350 3950 50  0001 C CNN
+F 3 "" H 4350 3950 50  0001 C CNN
+	1    4350 3950
+	1    0    0    -1
+$EndComp
+$Comp
+L +3V3 #PWR?
+U 1 1 5892A562
+P 4350 3500
+F 0 "#PWR?" H 4350 3350 50  0001 C CNN
+F 1 "+3V3" H 4350 3640 50  0000 C CNN
+F 2 "" H 4350 3500 50  0001 C CNN
+F 3 "" H 4350 3500 50  0001 C CNN
+	1    4350 3500
+	1    0    0    -1
+$EndComp
+$Comp
+L C C1d
+U 1 1 5892A578
+P 4350 3750
+F 0 "C1d" H 4200 3850 50  0000 L CNN
+F 1 "0.1uF" H 4150 3650 50  0000 L CNN
+F 2 "" H 4388 3600 50  0001 C CNN
+F 3 "" H 4350 3750 50  0001 C CNN
+	1    4350 3750
+	1    0    0    -1
+$EndComp
+Wire Wire Line
+	4350 3950 4350 3900
+Wire Wire Line
+	4350 3600 4350 3500
+Wire Wire Line
+	4850 3550 4350 3550
+Connection ~ 4350 3550
+$Comp
+L GND #PWR?
+U 1 1 5892A7AB
+P 6050 3650
+F 0 "#PWR?" H 6050 3400 50  0001 C CNN
+F 1 "GND" H 6050 3500 50  0000 C CNN
+F 2 "" H 6050 3650 50  0001 C CNN
+F 3 "" H 6050 3650 50  0001 C CNN
+	1    6050 3650
+	1    0    0    -1
+$EndComp
+Wire Wire Line
+	5700 3650 6050 3650
+Wire Wire Line
+	5700 2850 5750 2850
+Wire Wire Line
+	5750 2950 5700 2950
+Wire Wire Line
+	5700 3050 5750 3050
+Wire Wire Line
+	5750 3150 5700 3150
+Wire Wire Line
+	5750 3250 5700 3250
+Wire Wire Line
+	5750 3350 5700 3350
+Wire Wire Line
+	5750 3450 5700 3450
+Wire Wire Line
+	5700 3550 5750 3550
+Wire Wire Line
+	5750 3750 5700 3750
+Wire Wire Line
+	5750 3850 5700 3850
+Wire Wire Line
+	5750 3950 5700 3950
+Wire Wire Line
+	5750 4050 5700 4050
+Wire Wire Line
+	5750 4150 5700 4150
+Wire Wire Line
+	5750 4250 5700 4250
+Wire Wire Line
+	5750 4350 5700 4350
+Wire Wire Line
+	4800 4350 4850 4350
+Wire Wire Line
+	4850 4250 4800 4250
+Wire Wire Line
+	4850 4150 4800 4150
+Wire Wire Line
+	4850 4050 4800 4050
+Wire Wire Line
+	4850 3950 4800 3950
+Wire Wire Line
+	4850 3850 4800 3850
+Wire Wire Line
+	4850 3650 4800 3650
+Wire Wire Line
+	4800 3750 4850 3750
+Wire Wire Line
+	4850 3450 4800 3450
+Wire Wire Line
+	4800 3350 4850 3350
+Wire Wire Line
+	4850 3250 4800 3250
+Wire Wire Line
+	4800 3150 4850 3150
+Wire Wire Line
+	4850 3050 4800 3050
+Wire Wire Line
+	4800 2950 4850 2950
+Wire Wire Line
+	4850 2850 4800 2850
 $EndSCHEMATC
