File: design/electrical/microcontroller_module.sch (KiCad schematic (older format))
At the start: 0 parts

Commit message: Finished schematics
Parts:
- added C1c: 0.1uF, symbol C
- added C2c: 0.47uF, symbol C
- added P3a: CONN_01X06, symbol CONN_01X06
- added R1c: 4.75k, symbol R
- added R2c: 100k, symbol R
- added U2c: REF3130, symbol REF3130
- added U?: C8051F120, symbol C8051F120
Connections:
- net AIN0.0: now also U?.18 (AIN0.0)
- net AIN0.1: now also U?.19 (AIN0.1)
- net AIN0.2: now also U?.20 (AIN0.2)
- net AIN0.3: now also U?.21 (AIN0.3)
- net AIN0.4: now also U?.22 (AIN0.4)
- net AIN0.5: now also U?.23 (AIN0.5)
- net AIN0.6: now also U?.24 (AIN0.6)
- net AIN0.7: now also U?.25 (AIN0.7)
- net P0.0: now also U?.62 (P0.0)
- net P0.1: now also U?.61 (P0.1)
- net P0.2: now also U?.60 (P0.2)
- net P0.3: now also U?.59 (P0.3)
- net P0.4: now also U?.58 (P0.4)
- net P0.5: now also U?.57 (ALE/P0.5)
- net P0.6: now also U?.56 (/RD/P0.6)
- net P0.7: now also U?.55 (/WR/P0.7)
- net P1.0: now also U?.36 (AIN2.0/A8/P1.0)
- net P1.1: now also U?.35 (AIN2.1/A9/P1.1)
- net P1.2: now also U?.34 (AIN2.2/A10/P1.2)
- net P1.3: now also U?.33 (AIN2.3/A11/P1.3)
- net P1.4: now also U?.32 (AIN2.4/A12/P1.4)
- net P1.5: now also U?.31 (AIN2.5/A13/P1.5)
- net P1.6: now also U?.30 (AIN2.6/A14/P1.6)
- net P1.7: now also U?.29 (AIN2.7/A15/P1.7)
- net P2.0: now also U?.46 (A8m/A0/P2.0)
- net P2.1: now also U?.45 (A9m/A1/P2.1)
- net P2.2: now also U?.44 (A10m/A2/P2.2)
- net P2.3: now also U?.43 (A11m/A3/P2.3)
- net P2.4: now also U?.42 (A12m/A4/P2.4)
- net P2.5: now also U?.41 (A13m/A5/P2.5)
- net P2.6: now also U?.40 (A14m/A6/P2.6)
- net P2.7: now also U?.39 (A15m/A7/P2.7)
- net P3.0: now also U?.54 (AD0/D0/P3.0)
- net P3.1: now also U?.53 (AD1/D1/P3.1)
- net P3.2: now also U?.52 (AD2/D2/P3.2)
- net P3.3: now also U?.51 (AD3/D3/P3.3)
- net P3.4: now also U?.50 (AD4/D4/P3.4)
- net P3.5: now also U?.49 (AD5/D5/P3.5)
- net P3.6: now also U?.48 (AD6/D6/P3.6)
- net P3.7: now also U?.47 (AD7/D7/P3.7)
- net P4.0: now also U?.98 (P4.0)
- net P4.1: now also U?.97 (P4.1)
- net P4.2: now also U?.96 (P4.2)
- net P4.3: now also U?.95 (P4.3)
- net P4.4: now also U?.94 (P4.4)
- net P4.5: now also U?.93 (ALE/P4.5)
- net P4.6: now also U?.92 (/RD/P4.6)
- net P4.7: now also U?.91 (/WR/P4.7)
- net P5.0: now also U?.88 (A8/P5.0)
- net P5.1: now also U?.87 (A9/P5.1)
- net P5.2: now also U?.86 (A10/P5.2)
- net P5.3: now also U?.85 (A11/P5.3)
- net P5.4: now also U?.84 (A12/P5.4)
- net P5.5: now also U?.83 (A13/P5.5)
- net P5.6: now also U?.82 (A14/P5.6)
- net P5.7: now also U?.81 (A15/P5.7)
- net P6.0: now also U?.80 (A8m/A0/P6.0)
- net P6.1: now also U?.79 (A9m/A1/P6.1)
- net P6.2: now also U?.78 (A10m/A2/P6.2)
- net P6.3: now also U?.77 (A11m/A3/P6.3)
- net P6.4: now also U?.76 (A12m/A4/P6.4)
- net P6.5: now also U?.75 (A13m/A5/P6.5)
- net P6.6: now also U?.74 (A14m/A6/P6.6)
- net P6.7: now also U?.73 (A15m/A7/P6.7)
- net P7.0: now also U?.72 (AD0/D0/P7.0)
- net P7.1: now also U?.71 (AD1/D1/P7.1)
- net P7.2: now also U?.70 (AD2/D2/P7.2)
- net P7.3: now also U?.69 (AD3/D3/P7.3)
- net P7.4: now also U?.68 (AD4/D4/P7.4)
- net P7.5: now also U?.67 (AD5/D5/P7.5)
- net P7.6: now also U?.66 (AD6/D6/P7.6)
- net P7.7: now also U?.65 (AD7/D7/P7.7)
- new net: R2c.1, U?.5 (/RST)
- new net +3V3: C1c.2, C2c.1, P3a.1 (P1), R1c.1, R2c.2, U2c.1 (IN), U?.11 (AV+), U?.37 (VDD), U?.64 (VDD), U?.90 (VDD)
- new net GND: C1c.1, C2c.2, P3a.6 (P6), U2c.3 (GND), U?.10 (AGND), U?.13 (AGND), U?.28 (MONEN), U?.38 (DGND), U?.63 (DGND), U?.89 (DGND)
- new net TCK: P3a.3 (P3), R1c.2, U?.2 (TCK)
- new net TDI: P3a.4 (P4), U?.3 (TDI)
- new net TDO: P3a.5 (P5), U?.4 (TDO)
- new net TMS: P3a.2 (P2), U?.1 (TMS)
- new net VREF: U2c.2 (OUT), U?.15 (VREFD), U?.16 (VREF0), U?.17 (VREF2)
- no-connect marks 0 -> 10
