File: design/electrical/transceiver_module.sch (KiCad schematic (older format))
At the start: 0 parts

Commit message: Finished schematics
Parts:
- added C11e, C12e: 18pF, symbol C
- added C13e: 68pF, symbol C
- added C1e: 15pF, symbol C
- added C2e: 12pF, symbol C
- added C3e: 220pF, symbol C
- added C4e: 1uF, symbol C
- added C5e: 8.2pF, symbol C
- added C6e: 5.6pF, symbol C
- added C7e: 3.3uF, symbol C
- added C8e: 1nF, symbol C
- added C9e: 33nF, symbol C
- added L1e, L4e: BLM18HG102SN1D, symbol L
- added L2e: 68nH, symbol L
- added L3e: 6.2nH, symbol L
- added L5e: 33nH, symbol L
- added R1e: 10k, symbol R
- added R2e: 27k, symbol R
- added R3e: 82k, symbol R
- added U?: CC1000, TSSOP-28, symbol CC1000
- added Y1e: 14.7456MHz, symbol Crystal_GND2
Connections:
- net CHP_OUT: now also U?.12 (CHP_OUT)
- net RF_IN: now also C1e.1
- net RF_OUT: now also C6e.2
- net RSSI: now also C4e.1, R1e.2
- new net: L5e.2, U?.10 (L1)
- new net: L5e.1, U?.11 (L2)
- new net: R3e.1, U?.13 (R_BIAS)
- new net: C11e.1, U?.17 (XOSC_Q2), Y1e.3
- new net: C12e.1, U?.18 (XOSC_Q1), Y1e.1
- new net: L4e.2, U?.21 (DVDD)
- new net: R1e.1, R2e.1, U?.28 (RSSI/IF)
- new net: C1e.2, L2e.2, U?.3 (RF_IN)
- new net: C5e.1, C6e.1, L3e.1, U?.4 (RF_OUT)
- new net +3V3: L1e.1, L4e.1
- new net AVDD: C13e.1, C2e.1, C3e.1, C5e.2, C7e.1, C8e.1, C9e.1, L1e.2, L3e.2, U?.1 (AVDD), U?.15 (AVDD), U?.5 (AVDD), U?.9 (AVDD)
- new net GND: C11e.2, C12e.2, C13e.2, C2e.2, C3e.2, C4e.2, C7e.2, C8e.2, C9e.2, L2e.1, R2e.2, R3e.2, U?.14 (AGND), U?.16 (AGND), U?.19 (AGND), U?.2 (AGND), U?.20 (DGND), U?.22 (DGND), U?.6 (AGND), U?.7 (AGND), U?.8 (AGND), Y1e.2
Other:
- note added: "PIN 1"
- note added: "PIN 15"
- note added: "PIN 5"
- note added: "PIN 9"
